File: FabGL.kicad_pcb (KiCad board)
At the start: 2 copper layers, 65 x 56 mm, 254 parts, among them J2 Mini-DIN-6, J3 Mini-DIN-6, J6 DB15_Female_HighDensity, P1 2x40 2.54

Commit message: Pin swap
Fix pins so the board will boot, correction of error on use of strapping pins
Parts:
- added REF**: SolderWirePad_1x01_Drill0.8mm, Connector_Wire:SolderWirePad_1x01_Drill0.8mm, F.Cu at (138.8, 87.4)
- added REF**: SolderWirePad_1x01_Drill0.8mm, Connector_Wire:SolderWirePad_1x01_Drill0.8mm, F.Cu at (133.7, 79.9)
- added REF**: SolderWirePad_1x01_Drill0.8mm, Connector_Wire:SolderWirePad_1x01_Drill0.8mm, F.Cu at (136.2, 79.9)
- added REF**: SolderWirePad_1x01_Drill0.8mm, Connector_Wire:SolderWirePad_1x01_Drill0.8mm, F.Cu at (138.8, 79.9)
- added REF**: SolderWirePad_1x01_Drill0.8mm, Connector_Wire:SolderWirePad_1x01_Drill0.8mm, F.Cu at (141.0, 87.2)
- added REF**: SolderWirePad_1x01_Drill0.8mm, Connector_Wire:SolderWirePad_1x01_Drill0.8mm, F.Cu at (133.7, 87.4)
- added REF**: SolderWirePad_1x01_Drill0.8mm, Connector_Wire:SolderWirePad_1x01_Drill0.8mm, F.Cu at (131.2, 87.4)
- added REF**: SolderWirePad_1x01_Drill0.8mm, Connector_Wire:SolderWirePad_1x01_Drill0.8mm, F.Cu at (128.6, 87.4)
- added REF**: SolderWirePad_1x01_Drill0.8mm, Connector_Wire:SolderWirePad_1x01_Drill0.8mm, F.Cu at (136.2, 87.4)
- added REF**: SolderWirePad_1x01_Drill0.8mm, Connector_Wire:SolderWirePad_1x01_Drill0.8mm, F.Cu at (128.6, 79.9)
- added REF**: SolderWirePad_1x01_Drill0.8mm, Connector_Wire:SolderWirePad_1x01_Drill0.8mm, F.Cu at (126.4, 80.1)
- added REF**: SolderWirePad_1x01_Drill0.8mm, Connector_Wire:SolderWirePad_1x01_Drill0.8mm, F.Cu at (131.2, 79.9)
Connections:
- P1 pad 23: GREEN_LSB -> PS2_DAT
- P1 pad 35: PS2_DAT -> GREEN_LSB
Routing:
- net (no net): track 0.00 -> 22.2 mm
- net GREEN_LSB: track 28.2 -> 42.6 mm
- net PS2_DAT: track 2.72 -> 16.6 mm
